File: estop_remote_schematic/estop_remote_schematic.kicad_sch (KiCad schematic)
At the start: 18 parts, among them J1 Power Switch, J2 ESP32 Pins 1-22, J3 ESP32 Pins 23-44, J4 Battery Connector, J5 EStop Button, J6 OLed Screen Pins, J7 HC12 Connections, J8 Reset Button, J9 RotaryEnc Connections

Commit message: updated placements of SMD components to be more optimized for decoupling
Parts:
- J7: footprint Connector_PinHeader_2.54mm:PinHeader_1x05_P2.54mm_Vertical -> Connector_PinSocket_2.54mm:PinSocket_1x05_P2.54mm_Vertical
- renumbered HC12Capacitor1 to C1, HC12DecouplingCapacitor1 to C2, PowerCapacitor1 to C3, PowerCapacitor2 to C4, ADCDecouplingCapacitor1 to C5, I2CPullup1 to R1, I2CPullup2 to R2, VoltDivResistor1 to R3, VoltDivResistor2 to R4
Other:
- moved on the sheet: J4
Changed lines of the file:
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@@
 	(wire
 		(pts
-			(xy 71.12 27.94) (xy 71.12 34.29)
-		)
-		(stroke
-			(width 0)
-			(type default)
-		)
-	)
-	(wire
-		(pts
 			(xy 25.4 137.16) (xy 66.04 137.16)
 		)
@@
 	(wire
 		(pts
-			(xy 68.58 27.94) (xy 71.12 27.94)
+			(xy 68.58 27.94) (xy 74.93 27.94)
 		)
 		(stroke
@@
 	(wire
 		(pts
-			(xy 77.47 34.29) (xy 85.09 34.29)
+			(xy 77.47 27.94) (xy 85.09 27.94)
 		)
 		(stroke
@@
 	(wire
 		(pts
-			(xy 71.12 34.29) (xy 74.93 34.29)
-		)
-		(stroke
-			(width 0)
-			(type default)
-		)
-	)
-	(wire
-		(pts
 			(xy 36.83 160.02) (xy 66.04 160.02)
 		)
@@
 		(dnp no)
 		(fields_autoplaced yes)
-		(property "Reference" "I2CPullup1"
+		(property "Reference" "R1"
 			(at 35.56 186.6899 0)
 			(show_name no)
@@
 			(project "estop_remote_schematic"
 				(path "/5c08b7c6-3fe1-4a20-81ff-6cf06621ce55"
-					(reference "I2CPullup1")
+					(reference "R1")
 					(unit 1)
 				)
@@
 		(dnp no)
 		(fields_autoplaced yes)
-		(property "Reference" "ADCDecouplingCapacitor1"
+		(property "Reference" "C5"
 			(at 58.42 53.3399 0)
 			(show_name no)
@@
 			(project "estop_remote_schematic"
 				(path "/5c08b7c6-3fe1-4a20-81ff-6cf06621ce55"
-					(reference "ADCDecouplingCapacitor1")
+					(reference "C5")
 					(unit 1)
 				)
@@
 		(dnp no)
 		(property "Reference" "J1"
-			(at 68.072 26.67 90)
+			(at 73.406 30.734 90)
 			(show_name no)
 			(do_not_autoplace no)
@@
 		)
 		(property "Value" "Power Switch"
-			(at 73.914 24.13 90)
+			(at 84.074 33.02 90)
 			(show_name no)
 			(do_not_autoplace no)
@@
 		(dnp no)
 		(fields_autoplaced yes)
-		(property "Reference" "HC12DecouplingCapacitor1"
+		(property "Reference" "C2"
 			(at 59.69 129.5399 0)
 			(show_name no)
@@
 			(project "estop_remote_schematic"
 				(path "/5c08b7c6-3fe1-4a20-81ff-6cf06621ce55"
-					(reference "HC12DecouplingCapacitor1")
+					(reference "C2")
 					(unit 1)
 				)
@@
 		(dnp no)
 		(fields_autoplaced yes)
-		(property "Reference" "VoltDivResistor1"
+		(property "Reference" "R3"
 			(at 40.64 36.83 90)
 			(show_name no)
@@
 			(project "estop_remote_schematic"
 				(path "/5c08b7c6-3fe1-4a20-81ff-6cf06621ce55"
-					(reference "VoltDivResistor1")
+					(reference "R3")
 					(unit 1)
 				)
@@
 		(in_pos_files yes)
 		(dnp no)
-		(property "Reference" "PowerCapacitor2"
-			(at 17.272 28.448 0)
+		(property "Reference" "C4"
+			(at 29.464 29.21 0)
 			(show_name no)
 			(do_not_autoplace no)
@@
 			(project "estop_remote_schematic"
 				(path "/5c08b7c6-3fe1-4a20-81ff-6cf06621ce55"
-					(reference "PowerCapacitor2")
+					(reference "C4")
 					(unit 1)
 				)
@@
 		(dnp no)
 		(fields_autoplaced yes)
-		(property "Reference" "VoltDivResistor2"
+		(property "Reference" "R4"
 			(at 68.58 36.83 90)
 			(show_name no)
@@
 			(project "estop_remote_schematic"
 				(path "/5c08b7c6-3fe1-4a20-81ff-6cf06621ce55"
-					(reference "VoltDivResistor2")
+					(reference "R4")
 					(unit 1)
 				)
@@
 	(symbol
 		(lib_id "power:GND")
-		(at 85.09 34.29 90)
+		(at 85.09 27.94 90)
 		(unit 1)
 		(body_style 1)
@@
 		(fields_autoplaced yes)
 		(property "Reference" "#PWR02"
-			(at 91.44 34.29 0)
+			(at 91.44 27.94 0)
 			(hide yes)
 			(show_name no)
@@
 		)
 		(property "Value" "GND"
-			(at 88.9 34.2899 90)
+			(at 88.9 27.9399 90)
 			(show_name no)
 			(do_not_autoplace no)
@@
 		)
 		(property "Footprint" ""
-			(at 85.09 34.29 0)
+			(at 85.09 27.94 0)
 			(hide yes)
 			(show_name no)
@@
 		)
 		(property "Datasheet" ""
-			(at 85.09 34.29 0)
+			(at 85.09 27.94 0)
 			(hide yes)
 			(show_name no)
@@
 		)
 		(property "Description" "Power symbol creates a global label with name \"GND\" , ground"
-			(at 85.09 34.29 0)
+			(at 85.09 27.94 0)
 			(hide yes)
 			(show_name no)
@@
 		(in_pos_files yes)
 		(dnp no)
-		(property "Reference" "HC12Capacitor1"
-			(at 29.718 129.794 0)
+		(property "Reference" "C1"
+			(at 42.418 129.794 0)
 			(show_name no)
 			(do_not_autoplace no)
@@
 			(project "estop_remote_schematic"
 				(path "/5c08b7c6-3fe1-4a20-81ff-6cf06621ce55"
-					(reference "HC12Capacitor1")
+					(reference "C1")
 					(unit 1)
 				)
@@
 	(symbol
 		(lib_id "Connector_Generic:Conn_01x02")
-		(at 74.93 29.21 90)
+		(at 74.93 22.86 90)
 		(unit 1)
 		(body_style 1)
@@
 		(dnp no)
 		(property "Reference" "J4"
-			(at 79.502 27.94 90)
+			(at 79.502 21.59 90)
 			(show_name no)
 			(do_not_autoplace no)
@@
 		)
 		(property "Value" "Battery Connector"
-			(at 79.502 30.48 90)
+			(at 79.502 24.13 90)
 			(show_name no)
 			(do_not_autoplace no)
@@
 		)
 		(property "Footprint" "Connector_JST:JST_XH_B2B-XH-A_1x02_P2.50mm_Vertical"
-			(at 74.93 29.21 0)
+			(at 74.93 22.86 0)
 			(hide yes)
 			(show_name no)
@@
 		)
 		(property "Datasheet" ""
-			(at 74.93 29.21 0)
+			(at 74.93 22.86 0)
 			(hide yes)
 			(show_name no)
@@
 		)
 		(property "Description" "Generic connector, single row, 01x02, script generated (kicad-library-utils/schlib/autogen/connector/)"
-			(at 74.93 29.21 0)
+			(at 74.93 22.86 0)
 			(hide yes)
 			(show_name no)
@@
 		(dnp no)
 		(fields_autoplaced yes)
-		(property "Reference" "PowerCapacitor1"
+		(property "Reference" "C3"
 			(at 46.99 30.0989 0)
 			(show_name no)
@@
 			(project "estop_remote_schematic"
 				(path "/5c08b7c6-3fe1-4a20-81ff-6cf06621ce55"
-					(reference "PowerCapacitor1")
+					(reference "C3")
 					(unit 1)
 				)
@@
 			)
 		)
-		(property "Footprint" "Connector_PinHeader_2.54mm:PinHeader_1x05_P2.54mm_Vertical"
+		(property "Footprint" "Connector_PinSocket_2.54mm:PinSocket_1x05_P2.54mm_Vertical"
 			(at 71.12 137.16 0)
 			(hide yes)
@@
 		(dnp no)
 		(fields_autoplaced yes)
-		(property "Reference" "I2CPullup2"
+		(property "Reference" "R2"
 			(at 46.99 186.6899 0)
 			(show_name no)
@@
 			(project "estop_remote_schematic"
 				(path "/5c08b7c6-3fe1-4a20-81ff-6cf06621ce55"
-					(reference "I2CPullup2")
+					(reference "R2")
 					(unit 1)
 				)

Commit message: Modified values on components to be more standardized
Parts:
- removed J7: HC12 Connections, Connector_PinSocket_2.54mm:PinSocket_1x05_P2.54mm_Vertical, symbol Connector_Generic:Conn_01x05
- added J7: Conn_01x05_Socket, symbol Connector:Conn_01x05_Socket
- J1: value Power Switch -> JST-XH-2A
- J2: value ESP32 Pins 1-22 -> Conn_01x22
- J3: value ESP32 Pins 23-44 -> Conn_01x22
- J4: value Battery Connector -> JST-XH-2A
- J5: value EStop Button -> JST-XH-2A
- J6: value OLed Screen Pins -> Conn_01x04
- J8: value Reset Button -> JST-XH-2A
- J9: value RotaryEnc Connections -> JST-XH-5A
Connections:
- net +3.3V: now also J7.1 (Pin_1)
- net GND: now also J7.2 (Pin_2)
- net HC12_RX: now also J7.3 (Pin_3)
- net HC12_SET: now also J7.5 (Pin_5)
- net HC12_TX: now also J7.4 (Pin_4)
Other:
- note added: "Battery Connector"
- note added: "EStop Connector"
- note added: "HC-12 Connector"
- note added: "OLED Connector"
- note added: "Pins 1-22"
- note added: "Pins 23-44"
- note added: "Power Switch"
- note added: "Reset Connector"
- note added: "RotEnc Connector"
- moved on the sheet: J8
